File: compute/LoRaModule.sch (KiCad schematic (older format))
At the start: 28 parts

Commit message: small changes
Parts:
- U3: renamed from U?; symbol RF_SW:PE4259 -> g3_compute-rescue:PE4259-RF_SW
- gave numbers to parts that had none: 27

Commit message: Added interfacing to GPS Module
Parts:
- U2: symbol Transceivers:SX1262 -> g3_compute-rescue:SX1262-Transceivers
- U3: symbol g3_compute-rescue:PE4259-RF_SW -> g3_compute-rescue:PE4259-RF_SW-g3_compute-rescue
Changed lines of the file:
@@
 $EndDescr
 $Comp
-L Transceivers:SX1262 U2
+L g3_compute-rescue:SX1262-Transceivers U2
 U 1 1 6189FC0E
 P 4250 3450
+AR Path="/6189FC0E" Ref="U2"  Part="1"
+AR Path="/618967E8/6189FC0E" Ref="U2"  Part="1"
 F 0 "U2" H 4225 3925 50  0000 C CNN
 F 1 "SX1262" H 4225 3834 50  0000 C CNN
@@
 $EndComp
 $Comp
-L g3_compute-rescue:PE4259-RF_SW U3
+L g3_compute-rescue:PE4259-RF_SW-g3_compute-rescue U3
 U 1 1 618EAA8C
 P 8750 3650
