File: compute/SX1262LoRaModule.sch (KiCad schematic (older format))
At the start: 28 parts, among them U201 SX1262, U202 PE4259, Y201 TBD

Commit message: Updated BOM
Parts:
- C203: Description (none) -> 1uF Capacitor; MFN (none) -> Yageo; MFP (none) -> CC0402MRX5R6BB105; Notes DNL -> (none); S1PL https://www.digikey.com/en/products/detail/samsung-electro-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 -> https://www.digikey.com/en/products/detail/yageo/CC0402MRX5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; S1PN Digikey -> 311-1732; S2PL (none) -> https://www.mouser.com/ProductDetail/YAGEO/CC0402MRX5R6BB10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; S2PN (none) -> 603-CC402MRX5R6BB105
Changed lines of the file:
@@
 F 1 "1uF" H 3465 2855 50  0000 L CNN
 F 2 "Capacitor_SMD:C_0402_1005Metric_Pad0.74x0.62mm_HandSolder" H 3388 2750 50  0001 C CNN
-F 3 "~" H 3350 2900 50  0001 C CNN
-F 4 "" H 3350 2900 50  0001 C CNN "MFN"
-F 5 "" H 3350 2900 50  0001 C CNN "MFP"
-F 6 "Digikey" H 3350 2900 50  0001 C CNN "S1PN"
-F 7 "https://www.digikey.com/en/products/detail/samsung-electro-mechanics/CL05B103KO5NNNC/3886709" H 3350 2900 50  0001 C CNN "S1PL"
-F 8 "DNL" H 3350 2900 50  0001 C CNN "Notes"
+F 3 "https://www.yageo.com/upload/media/product/productsearch/datasheet/mlcc/UPY-GPHC_X5R_4V-to-50V_26.pdf" H 3350 2900 50  0001 C CNN
+F 4 "Yageo" H 3350 2900 50  0001 C CNN "MFN"
+F 5 "CC0402MRX5R6BB105" H 3350 2900 50  0001 C CNN "MFP"
+F 6 "311-1732" H 3350 2900 50  0001 C CNN "S1PN"
+F 7 "https://www.digikey.com/en/products/detail/yageo/CC0402MRX5R6BB105/5195141" H 3350 2900 50  0001 C CNN "S1PL"
+F 8 "" H 3350 2900 50  0001 C CNN "Notes"
+F 9 "1uF Capacitor" H 3350 2900 50  0001 C CNN "Description"
+F 10 "https://www.mouser.com/ProductDetail/YAGEO/CC0402MRX5R6BB105?qs=sGAEpiMZZMt1iCLsaqcCFv92tuvmRjoeIh9ul0L8pvU%3D" H 3350 2900 50  0001 C CNN "S2PL"
+F 11 "603-CC402MRX5R6BB105" H 3350 2900 50  0001 C CNN "S2PN"
 	1    3350 2900
 	1    0    0    -1

Commit message: First alternative revision
Connections:
- net ANT: no longer C215.1, U202.5 (RFC)
- net at L203.1, U201.22 (RFI_N): now also C208.1
- net at C206.1, L203.2, U201.21 (RFI_P): no longer C208.1
- new net: C215.1, U202.5 (RFC)
Other:
- moved on the sheet: C206, C208, C210, L203
Changed lines of the file:
@@
 L Device:L L203
 U 1 1 618C8BAD
-P 5850 4150
+P 6025 4425
 AR Path="/624C3AFD/618C8BAD" Ref="L203"  Part="1"
 AR Path="/61FFC2A4/618C8BAD" Ref="L?"  Part="1"
-F 0 "L203" V 6040 4150 50  0000 C CNN
-F 1 "15nH" V 5949 4150 50  0000 C CNN
-F 2 "Inductor_SMD:L_0402_1005Metric_Pad0.77x0.64mm_HandSolder" H 5850 4150 50  0001 C CNN
-F 3 "~" H 5850 4150 50  0001 C CNN
-F 4 "" V 5850 4150 50  0001 C CNN "MFN"
-F 5 "" V 5850 4150 50  0001 C CNN "MFP"
-F 6 "" V 5850 4150 50  0001 C CNN "S1PN"
-F 7 "" V 5850 4150 50  0001 C CNN "S1PL"
-F 8 "DNL" V 5850 4150 50  0001 C CNN "Notes"
-	1    5850 4150
+F 0 "L203" V 6215 4425 50  0000 C CNN
+F 1 "15nH" V 6124 4425 50  0000 C CNN
+F 2 "Inductor_SMD:L_0402_1005Metric_Pad0.77x0.64mm_HandSolder" H 6025 4425 50  0001 C CNN
+F 3 "~" H 6025 4425 50  0001 C CNN
+F 4 "" V 6025 4425 50  0001 C CNN "MFN"
+F 5 "" V 6025 4425 50  0001 C CNN "MFP"
+F 6 "" V 6025 4425 50  0001 C CNN "S1PN"
+F 7 "" V 6025 4425 50  0001 C CNN "S1PL"
+F 8 "DNL" V 6025 4425 50  0001 C CNN "Notes"
+	1    6025 4425
 	1    0    0    -1
 $EndComp
 Wire Wire Line
 	4800 3400 5850 3400
-Wire Wire Line
-	5850 3400 5850 4000
 Wire Wire Line
 	4800 3500 5700 3500
@@
 L Device:C C206
 U 1 1 618CE91A
-P 5850 4650
+P 6025 4900
 AR Path="/624C3AFD/618CE91A" Ref="C206"  Part="1"
 AR Path="/61FFC2A4/618CE91A" Ref="C?"  Part="1"
-F 0 "C206" H 5965 4696 50  0000 L CNN
-F 1 "1.8pF" H 5965 4605 50  0000 L CNN
-F 2 "Capacitor_SMD:C_0402_1005Metric_Pad0.74x0.62mm_HandSolder" H 5888 4500 50  0001 C CNN
-F 3 "~" H 5850 4650 50  0001 C CNN
-F 4 "" H 5850 4650 50  0001 C CNN "MFN"
-F 5 "" H 5850 4650 50  0001 C CNN "MFP"
-F 6 "" H 5850 4650 50  0001 C CNN "S1PN"
-F 7 "" H 5850 4650 50  0001 C CNN "S1PL"
-F 8 "DNL" H 5850 4650 50  0001 C CNN "Notes"
-	1    5850 4650
-	1    0    0    -1
-$EndComp
-Wire Wire Line
-	5850 4300 5850 4350
-Wire Wire Line
-	5700 4350 5850 4350
-Wire Wire Line
-	5700 3500 5700 4350
-Connection ~ 5850 4350
+F 0 "C206" H 6140 4946 50  0000 L CNN
+F 1 "1.8pF" H 6140 4855 50  0000 L CNN
+F 2 "Capacitor_SMD:C_0402_1005Metric_Pad0.74x0.62mm_HandSolder" H 6063 4750 50  0001 C CNN
+F 3 "~" H 6025 4900 50  0001 C CNN
+F 4 "" H 6025 4900 50  0001 C CNN "MFN"
+F 5 "" H 6025 4900 50  0001 C CNN "MFP"
+F 6 "" H 6025 4900 50  0001 C CNN "S1PN"
+F 7 "" H 6025 4900 50  0001 C CNN "S1PL"
+F 8 "DNL" H 6025 4900 50  0001 C CNN "Notes"
+	1    6025 4900
+	1    0    0    -1
+$EndComp
 $Comp
 L power:GND #PWR0209
 U 1 1 618D373E
-P 5850 4800
+P 6025 5050
 AR Path="/624C3AFD/618D373E" Ref="#PWR0209"  Part="1"
 AR Path="/61FFC2A4/618D373E" Ref="#PWR?"  Part="1"
-F 0 "#PWR0209" H 5850 4550 50  0001 C CNN
-F 1 "GND" H 5855 4627 50  0000 C CNN
-F 2 "" H 5850 4800 50  0001 C CNN
-F 3 "" H 5850 4800 50  0001 C CNN
-	1    5850 4800
+F 0 "#PWR0209" H 6025 4800 50  0001 C CNN
+F 1 "GND" H 6030 4877 50  0000 C CNN
+F 2 "" H 6025 5050 50  0001 C CNN
+F 3 "" H 6025 5050 50  0001 C CNN
+	1    6025 5050
 	1    0    0    -1
 $EndComp
@@
 L Device:C C208
 U 1 1 618D3CBD
-P 6300 4400
+P 6550 4225
 AR Path="/624C3AFD/618D3CBD" Ref="C208"  Part="1"
 AR Path="/61FFC2A4/618D3CBD" Ref="C?"  Part="1"
-F 0 "C208" H 6415 4446 50  0000 L CNN
-F 1 "2.4pF" H 6415 4355 50  0000 L CNN
-F 2 "Capacitor_SMD:C_0402_1005Metric_Pad0.74x0.62mm_HandSolder" H 6338 4250 50  0001 C CNN
-F 3 "~" H 6300 4400 50  0001 C CNN
-F 4 "" H 6300 4400 50  0001 C CNN "MFN"
-F 5 "" H 6300 4400 50  0001 C CNN "MFP"
-F 6 "Digikey" H 6300 4400 50  0001 C CNN "S1PN"
-F 7 "https://www.digikey.com/en/products/detail/taiyo-yuden/EVK105CH0R3BW-F/1169601" H 6300 4400 50  0001 C CNN "S1PL"
-F 8 "DNL" H 6300 4400 50  0001 C CNN "Notes"
-	1    6300 4400
+F 0 "C208" V 6400 4125 50  0000 L CNN
+F 1 "2.4pF" V 6325 4100 50  0000 L CNN
+F 2 "Capacitor_SMD:C_0402_1005Metric_Pad0.74x0.62mm_HandSolder" H 6588 4075 50  0001 C CNN
+F 3 "~" H 6550 4225 50  0001 C CNN
+F 4 "" H 6550 4225 50  0001 C CNN "MFN"
+F 5 "" H 6550 4225 50  0001 C CNN "MFP"
+F 6 "Digikey" H 6550 4225 50  0001 C CNN "S1PN"
+F 7 "https://www.digikey.com/en/products/detail/taiyo-yuden/EVK105CH0R3BW-F/1169601" H 6550 4225 50  0001 C CNN "S1PL"
+F 8 "DNL" H 6550 4225 50  0001 C CNN "Notes"
+	1    6550 4225
 	0    -1   -1   0
 $EndComp
@@
 L Device:C C210
 U 1 1 618D4647
-P 6700 4550
+P 7050 4375
 AR Path="/624C3AFD/618D4647" Ref="C210"  Part="1"
 AR Path="/61FFC2A4/618D4647" Ref="C?"  Part="1"
-F 0 "C210" H 6815 4596 50  0000 L CNN
-F 1 "4.7pF" H 6815 4505 50  0000 L CNN
-F 2 "Capacitor_SMD:C_0402_1005Metric_Pad0.74x0.62mm_HandSolder" H 6738 4400 50  0001 C CNN
-F 3 "~" H 6700 4550 50  0001 C CNN
-F 4 "" H 6700 4550 50  0001 C CNN "MFN"
-F 5 "" H 6700 4550 50  0001 C CNN "MFP"
-F 6 "" H 6700 4550 50  0001 C CNN "S1PN"
-F 7 "" H 6700 4550 50  0001 C CNN "S1PL"
-F 8 "DNL" H 6700 4550 50  0001 C CNN "Notes"
-	1    6700 4550
-	1    0    0    -1
-$EndComp
-Wire Wire Line
-	5850 4350 5850 4400
-Wire Wire Line
-	5850 4400 6150 4400
-Connection ~ 5850 4400
-Wire Wire Line
-	5850 4400 5850 4500
-Wire Wire Line
-	6450 4400 6700 4400
+F 0 "C210" H 7165 4421 50  0000 L CNN
+F 1 "4.7pF" H 7165 4330 50  0000 L CNN
+F 2 "Capacitor_SMD:C_0402_1005Metric_Pad0.74x0.62mm_HandSolder" H 7088 4225 50  0001 C CNN
+F 3 "~" H 7050 4375 50  0001 C CNN
+F 4 "" H 7050 4375 50  0001 C CNN "MFN"
+F 5 "" H 7050 4375 50  0001 C CNN "MFP"
+F 6 "" H 7050 4375 50  0001 C CNN "S1PN"
+F 7 "" H 7050 4375 50  0001 C CNN "S1PL"
+F 8 "DNL" H 7050 4375 50  0001 C CNN "Notes"
+	1    7050 4375
+	1    0    0    -1
+$EndComp
 $Comp
 L power:GND #PWR0211
 U 1 1 618DD2D6
-P 6700 4700
+P 7050 4525
 AR Path="/624C3AFD/618DD2D6" Ref="#PWR0211"  Part="1"
 AR Path="/61FFC2A4/618DD2D6" Ref="#PWR?"  Part="1"
-F 0 "#PWR0211" H 6700 4450 50  0001 C CNN
-F 1 "GND" H 6705 4527 50  0000 C CNN
-F 2 "" H 6700 4700 50  0001 C CNN
-F 3 "" H 6700 4700 50  0001 C CNN
-	1    6700 4700
-	1    0    0    -1
-$EndComp
-Wire Wire Line
-	6700 4400 8050 4400
-Connection ~ 6700 4400
+F 0 "#PWR0211" H 7050 4275 50  0001 C CNN
+F 1 "GND" H 7055 4352 50  0000 C CNN
+F 2 "" H 7050 4525 50  0001 C CNN
+F 3 "" H 7050 4525 50  0001 C CNN
+	1    7050 4525
+	1    0    0    -1
+$EndComp
 Wire Wire Line
 	8050 3300 8050 3850
 Wire Wire Line
 	8050 3850 8350 3850
-Wire Wire Line
-	8050 4400 8050 4050
 Wire Wire Line
 	8350 4050 8050 4050
@@
 	1    0    0    -1
 $EndComp
-Text Label 9100 3950 0    50   ~ 0
-ANT
 $Comp
 L Device:L L201
@@
 Wire Wire Line
 	3650 3400 3075 3400
+Wire Wire Line
+	6700 4225 7050 4225
+Wire Wire Line
+	8050 4225 8050 4050
+Connection ~ 7050 4225
+Wire Wire Line
+	7050 4225 8050 4225
+Wire Wire Line
+	5850 3400 5850 4225
+Wire Wire Line
+	5850 4225 6025 4225
+Connection ~ 6025 4225
+Wire Wire Line
+	6025 4225 6400 4225
+Wire Wire Line
+	6025 4225 6025 4275
+Wire Wire Line
+	5700 3500 5700 4625
+Wire Wire Line
+	6025 4625 6025 4750
+Wire Wire Line
+	6025 4625 6025 4575
+Connection ~ 6025 4625
+Wire Wire Line
+	5700 4625 6025 4625
 $EndSCHEMATC
